File: Minor Projects/JukeboxRelay/LatchRelay.sch (KiCad schematic (older format))
At the start: 7 parts, among them Q1 Q_NPN_BCE, Q2 Q_NPN_BCE

Commit message: Finished Jukebox Relay Design
Parts:
- removed Q1, Q2: Q_NPN_BCE, symbol Q_NPN_BCE
- removed Q?: Q_NMOS_DGS, symbol Q_NMOS_DGS
- removed R? (x4): R, symbol R
- added D1, D2: LED_Small, LEDs:LED_D4.0mm, symbol device:LED_Small
- added J1: Relay Socket, Library:Terminal_Block_Relay, symbol conn:Conn_01x10_Male
- added K1: AZ850P2-x, Library:Relay, symbol relay:AZ850P2-x
- added R1: 500, Library:42J500E, symbol device:R
- added R2: 390, Library:FMP200JR-52-390R, symbol device:R
Connections:
- net labels removed: GND, VCC
- wire segments 13 -> 48
Other:
- note added: "Jukebox Relay Replacement"
