File: Minor Projects/SpaceInvadersHeadboard/HeadboardDriver.sch (KiCad schematic (older format))
At the start: 11 parts, among them Q1 Q_NMOS_DGS, Q2 Q_NMOS_DGS, Q3 Q_NMOS_DGS, Q4 Q_NMOS_DGS, U1 NE555, U2 74LS76, U3 74LS08

Commit message: Completed JukeBox and SpaceInvader PCBs Created Gerbers Ordered Parts
Parts:
- removed LA1, LA2, LA3, LA4: Lamp, symbol Lamp
- removed Q1, Q2, Q3, Q4: Q_NMOS_DGS, symbol Q_NMOS_DGS
- removed U1: NE555, symbol NE555
- removed U2: 74LS76, symbol 74LS76
- removed U3: 74LS08, symbol 74LS08
- added C1: 0.01u, Capacitors_SMD:C_0805_HandSoldering, symbol device:C
- added C2: 10u, Capacitors_SMD:C_0805_HandSoldering, symbol device:C
- added D1: MUR2100ERLGOSCT-ND, Diodes_THT:D_DO-41_SOD81_P10.16mm_Horizontal, symbol device:D
- added J1: Loads, Library:640456-7, symbol conn:Conn_01x07_Female
- added J2: Conn_Coaxial_Power, Connectors:BARREL_JACK, symbol conn:Conn_Coaxial_Power
- added K1, K2: RELAYNLT, Library:EC2-5NU, symbol EC2-5NU:RELAYNLT
- added Q1, Q2: 2N7000TACT-ND, TO_SOT_Packages_THT:TO-92_Inline_Wide, symbol device:Q_NMOS_DGS
- added R1: 5.6k, Resistors_THT:R_Axial_DIN0207_L6.3mm_D2.5mm_P10.16mm_Horizontal, symbol device:R
- added R2: 33k, Resistors_THT:R_Axial_DIN0207_L6.3mm_D2.5mm_P10.16mm_Horizontal, symbol device:R
- added U1: CD40193BE, Library:CD40193BE, symbol CD40193BE:CD40193BE
- added U2: LM555, Housings_DIP:DIP-8_W7.62mm, symbol linear:LM555
Connections:
- net labels added: 0, A, B, C, C1, C2, D, Vcc, X, Y
- net labels removed: GND, VCC
- wire segments 64 -> 96
Other:
- note added: "10V"
- note added: "10V 2A"
- note added: "12V 2.5A"
